File: pcb/marlin_interface.brd (EAGLE design)
At the start: 28.9 x 29.2 mm, 8 parts

Commit message: remove auto mode from sd
Connections:
- net N$12: no longer U$1.JP2.3
Changed lines of the file:
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@@
 </signal>
 <signal name="N$12">
-<contactref element="U$1" pad="JP2.3"/>
 <contactref element="R6" pad="1"/>
 <contactref element="U$1" pad="JP2.4"/>
@@
 <wire x1="26.5" y1="19" x2="26.67" y2="19.05" width="0.6" layer="1"/>
 <wire x1="24" y1="19" x2="26.5" y2="21.5" width="0.6" layer="1"/>
-<wire x1="26.5" y1="21.5" x2="26.67" y2="21.59" width="0.6" layer="1"/>
 </signal>
 <signal name="N$13">
